File: s88isolated/s88iso/s88iso.sch (KiCad schematic (older format))
At the start: 26 parts, among them J1 Barrel_Jack_Switch_MountingPin, J2 5V Bypass, J3 12V 5V, J4 Conn_01x04, U1 L7805, U2 4504, U3 Si8641BB-B

Commit message: new V2.0 version for JLCPCB Assembly Service
Parts:
- removed C5: 1nF, Capacitor_SMD:C_0805_2012Metric, symbol Device:C
- removed U1: L7805, Package_TO_SOT_SMD:TO-252-2, symbol Regulator_Linear:L7805
- added D1: M7, Diode_SMD:D_SMA, symbol Device:D
- added D2: Power LED, LED_SMD:LED_0603_1608Metric_Pad1.05x0.95mm_HandSolder, symbol Device:LED
- added D3: 5V1, Diode_SMD:D_0805_2012Metric_Pad1.15x1.40mm_HandSolder, symbol Device:D_Zener
- added R10: 1k, Resistor_SMD:R_0603_1608Metric_Pad0.98x0.95mm_HandSolder, symbol Device:R
- added U1: LM317, Package_TO_SOT_SMD:TO-252-2, symbol Regulator_Linear:LM317_TO-252
- C1, C3, C4, C6, C7: LCSC (none) -> C28233
- C2: value 100nF -> 1uF; footprint Capacitor_SMD:C_0805_2012Metric -> Capacitor_SMD:C_0805_2012Metric_Pad1.18x1.45mm_HandSolder; LCSC (none) -> C28323
- R1: value 47 -> 240; footprint Resistor_SMD:R_0805_2012Metric -> Resistor_SMD:R_0603_1608Metric_Pad0.98x0.95mm_HandSolder; LCSC (none) -> C23350
- R2: value 47 -> 750; footprint Resistor_SMD:R_0805_2012Metric -> Resistor_SMD:R_0603_1608Metric_Pad0.98x0.95mm_HandSolder; LCSC (none) -> C23241
- R3: value 47 -> 270; footprint Resistor_SMD:R_0805_2012Metric -> Resistor_SMD:R_0603_1608Metric_Pad0.98x0.95mm_HandSolder; LCSC (none) -> C22966
- R4: LCSC (none) -> C4310
- R5: LCSC (none) -> C25804
- R6, R7, R8: value 47 -> 56; footprint Resistor_SMD:R_0805_2012Metric -> Resistor_SMD:R_0603_1608Metric_Pad0.98x0.95mm_HandSolder; LCSC (none) -> C25196
- R9: value 47 -> 1k; footprint Resistor_SMD:R_0805_2012Metric -> Resistor_SMD:R_0603_1608Metric_Pad0.98x0.95mm_HandSolder; LCSC (none) -> C21190
- U2: footprint w_smd_dil:so-16 -> Package_SO:SOIC-16_3.9x9.9mm_P1.27mm; LCSC (none) -> C151885
- U3: value Si8641BB-B -> NSI8141W1; footprint w_smd_dil:so-16 -> Package_SO:SOIC-16W_7.5x10.3mm_P1.27mm; LCSC (none) -> C399514
Connections:
- wire segments 125 -> 134
Other:
- moved on the sheet: C1, C6, C7, J1, J2, J3

Commit message: fix LED
Parts:
- D2: LCSC C2286 -> C72043
Changed lines of the file:
@@
 F 2 "LED_SMD:LED_0603_1608Metric_Pad1.05x0.95mm_HandSolder" H 6225 2100 50  0001 C CNN
 F 3 "~" H 6225 2100 50  0001 C CNN
-F 4 "C2286" V 6225 2100 50  0001 C CNN "LCSC"
+F 4 "C72043" V 6225 2100 50  0001 C CNN "LCSC"
 	1    6225 2100
 	0    -1   -1   0
